Commit message: Created simple tilt_servo macro in multirotor_base and removed controller_interface from firefly_base
- tilt_servo is a position controlled motor
- firefly_tilt.xacro contains an example of how to add a tilt servo

- Since controller interface plugin is not fully implemented yet, bypassed commandSubTopic in vertical_rotor macro

File: rotors_description/urdf/firefly_base.xacro (robot description, xacro)
@@ -21,5 +21,5 @@
   <xacro:include filename="$(find rotors_description)/urdf/firefly.xacro" />
   <!-- Instantiate a controller. -->
-  <xacro:controller_plugin_macro namespace="${namespace}" imu_sub_topic="imu" />
+<!--  <xacro:controller_plugin_macro namespace="${namespace}" imu_sub_topic="imu" />-->
   <!-- Instantiate a ROS message interface -->
   <!-- <xacro:ros_interface_plugin_macro namespace="${namespace}" />-->

File: rotors_description/urdf/multirotor_base.xacro (robot description, xacro)
@@ -120,5 +120,5 @@
         <motorConstant>${motor_constant}</motorConstant>
         <momentConstant>${moment_constant}</momentConstant>
-        <commandSubTopic>gazebo/command/motor_speed</commandSubTopic>
+        <commandSubTopic>command/motor_speed</commandSubTopic>
         <motorNumber>${motor_number}</motorNumber>
         <rotorDragCoefficient>${rotor_drag_coefficient}</rotorDragCoefficient>
@@ -132,3 +132,56 @@
     </gazebo>
   </xacro:macro>
+ <!-- Tilt servo joint and link (isolated from rotor command)-->
+  <xacro:macro name="tilt_servo"
+    params="robot_namespace suffix direction parent link_mass link_length link_radius motor_number color use_own_mesh mesh kp kd *origin *axis *inertia">
+    <joint name="${robot_namespace}/tilt_${motor_number}_joint" type="continuous">
+      <xacro:insert_block name="origin" />
+      <xacro:insert_block name="axis" />
+      <parent link="${parent}" />
+      <child link="${robot_namespace}/tilt_${motor_number}" />
+    </joint>
+    <link name="${robot_namespace}/tilt_${motor_number}">
+      <inertial>
+        <mass value="${link_mass}" /> <!-- [kg] -->
+        <xacro:insert_block name="inertia" />
+      </inertial>
+      <visual>
+        <geometry>
+          <!-- <cylinder length="0.005" radius="${radius_rotor}"/> --> <!-- [m] -->
+          <xacro:if value="${use_own_mesh}">
+            <mesh filename="${mesh}"
+              scale="1 1 1" />
+          </xacro:if>
+          <xacro:unless value="${use_own_mesh}">
+            <cylinder length="${link_length}" radius="${link_radius}"/> <!-- [m] -->
+          </xacro:unless>
+        </geometry>
+      </visual>
+<!--      <collision>
+        <geometry>
+          <cylinder length="${link_length}" radius="${link_radius}" />
+        </geometry>
+      </collision>-->
+    </link>
+    <gazebo>
+      <plugin name="${robot_namespace}_${suffix}_tilt_servo" filename="librotors_gazebo_motor_model.so">
+        <robotNamespace>${robot_namespace}</robotNamespace>
+        <jointName>${robot_namespace}/tilt_${motor_number}_joint</jointName>
+        <linkName>${robot_namespace}/tilt_${motor_number}</linkName>
+        <turningDirection>${direction}</turningDirection>
+        <motorType>position</motorType>
+        <joint_control_pid>
+            <p>${kp}</p>
+            <d>${kd}</d>
+        </joint_control_pid>
+        <commandSubTopic>command/tilt_pos</commandSubTopic>
+        <motorNumber>${motor_number}</motorNumber>
+        <motorSpeedPubTopic>tilt_speed/${motor_number}</motorSpeedPubTopic>
+        <motorPositionPubTopic>tilt_pos/${motor_number}</motorPositionPubTopic>
+      </plugin>
+    </gazebo>
+    <gazebo reference="${robot_namespace}/tilt_${motor_number}">
+      <material>Gazebo/${color}</material>
+    </gazebo>
+  </xacro:macro>
 </robot>
