Commit message: Added ball_joint and suspended_load macros in multirotor_base.xacro
- Firefly is temporarily modified with a suspended load
- The cable might have multiple links. It works well up to five links

File: rotors_description/urdf/firefly.urdf (robot description, URDF)
Before this commit: robot firefly, 11 links, 10 joints
Links:
- removed link firefly/cable_link_0a
- removed link firefly/cable_link_0b
- removed link firefly/cable_load_link
- added link firefly/cable_joint_0_link, mass 1e-14
- added link firefly/cable_joint_1_link, mass 1e-14
- added link firefly/cable_joint_2_link, mass 1e-14
- added link firefly/cable_joint_3_link, mass 1e-14
- added link firefly/cable_joint_4_link, mass 1e-14
- added link firefly/cable_joint_5_link, mass 1e-14
- added link firefly/cable_joint_6_link, mass 1e-14
- added link firefly/cable_joint_7_link, mass 1e-14
- added link firefly/cable_joint_8_link, mass 1e-14
- added link firefly/cable_joint_9_link, mass 1e-14
- added link firefly/cable_link_0, mass 0.0005; visual cylinder length=0.1 radius=0.005
- added link firefly/cable_link_1, mass 0.0005; visual cylinder length=0.1 radius=0.005
- added link firefly/cable_link_2, mass 0.0005; visual cylinder length=0.1 radius=0.005
- added link firefly/cable_link_3, mass 0.0005; visual cylinder length=0.1 radius=0.005
- added link firefly/cable_link_4, mass 0.0005; visual cylinder length=0.1 radius=0.005
- added link firefly/cable_link_5, mass 0.0005; visual cylinder length=0.1 radius=0.005
- added link firefly/cable_link_6, mass 0.0005; visual cylinder length=0.1 radius=0.005
- added link firefly/cable_link_7, mass 0.0005; visual cylinder length=0.1 radius=0.005
- added link firefly/cable_link_8, mass 0.0005; visual cylinder length=0.1 radius=0.005
- added link firefly/cable_link_9, mass 0.0005; visual cylinder length=0.1 radius=0.005
- added link firefly/load_cable_joint_link, mass 1e-14
- added link firefly/load_link, mass 0.2; visual sphere radius=0.05
Joints:
- removed joint firefly/cable_joint_0a
- removed joint firefly/cable_joint_0b
- removed joint firefly/cable_load_joint
- added joint firefly/cable_joint_0: type continuous, parent firefly/cable_joint_0_link, child firefly/cable_link_0, axis 0 1 0
- added joint firefly/cable_joint_0_aux: type continuous, parent firefly/base_link, child firefly/cable_joint_0_link, origin xyz=0 0 0 rpy=0 0 0, axis 1 0 0
- added joint firefly/cable_joint_1: type continuous, parent firefly/cable_joint_1_link, child firefly/cable_link_1, axis 0 1 0
- added joint firefly/cable_joint_1_aux: type continuous, parent firefly/cable_link_0, child firefly/cable_joint_1_link, origin xyz=0 0 -0.1, axis 1 0 0
- added joint firefly/cable_joint_2: type continuous, parent firefly/cable_joint_2_link, child firefly/cable_link_2, axis 0 1 0
- added joint firefly/cable_joint_2_aux: type continuous, parent firefly/cable_link_1, child firefly/cable_joint_2_link, origin xyz=0 0 -0.1, axis 1 0 0
- added joint firefly/cable_joint_3: type continuous, parent firefly/cable_joint_3_link, child firefly/cable_link_3, axis 0 1 0
- added joint firefly/cable_joint_3_aux: type continuous, parent firefly/cable_link_2, child firefly/cable_joint_3_link, origin xyz=0 0 -0.1, axis 1 0 0
- added joint firefly/cable_joint_4: type continuous, parent firefly/cable_joint_4_link, child firefly/cable_link_4, axis 0 1 0
- added joint firefly/cable_joint_4_aux: type continuous, parent firefly/cable_link_3, child firefly/cable_joint_4_link, origin xyz=0 0 -0.1, axis 1 0 0
- added joint firefly/cable_joint_5: type continuous, parent firefly/cable_joint_5_link, child firefly/cable_link_5, axis 0 1 0
- added joint firefly/cable_joint_5_aux: type continuous, parent firefly/cable_link_4, child firefly/cable_joint_5_link, origin xyz=0 0 -0.1, axis 1 0 0
- added joint firefly/cable_joint_6: type continuous, parent firefly/cable_joint_6_link, child firefly/cable_link_6, axis 0 1 0
- added joint firefly/cable_joint_6_aux: type continuous, parent firefly/cable_link_5, child firefly/cable_joint_6_link, origin xyz=0 0 -0.1, axis 1 0 0
- added joint firefly/cable_joint_7: type continuous, parent firefly/cable_joint_7_link, child firefly/cable_link_7, axis 0 1 0
- added joint firefly/cable_joint_7_aux: type continuous, parent firefly/cable_link_6, child firefly/cable_joint_7_link, origin xyz=0 0 -0.1, axis 1 0 0
- added joint firefly/cable_joint_8: type continuous, parent firefly/cable_joint_8_link, child firefly/cable_link_8, axis 0 1 0
- added joint firefly/cable_joint_8_aux: type continuous, parent firefly/cable_link_7, child firefly/cable_joint_8_link, origin xyz=0 0 -0.1, axis 1 0 0
- added joint firefly/cable_joint_9: type continuous, parent firefly/cable_joint_9_link, child firefly/cable_link_9, axis 0 1 0
- added joint firefly/cable_joint_9_aux: type continuous, parent firefly/cable_link_8, child firefly/cable_joint_9_link, origin xyz=0 0 -0.1, axis 1 0 0
- added joint firefly/load_cable_joint: type continuous, parent firefly/load_cable_joint_link, child firefly/load_link, axis 0 1 0
- added joint firefly/load_cable_joint_aux: type continuous, parent firefly/cable_link_9, child firefly/load_cable_joint_link, origin xyz=0 0 -0.1, axis 1 0 0

File: rotors_description/urdf/firefly.xacro (robot description, xacro)
@@ -184,23 +184,18 @@
     <xacro:insert_block name="rotor_inertia" />
   </xacro:vertical_rotor>
-  <xacro:vertical_cable
-    robot_namespace="${namespace}"
-    parent="${namespace}/base_link"
-    number_of_links="1"
-    link_length="0.5"
+  <xacro:suspended_load
+    robot_namespace="${namespace}"
+    parent="${namespace}/base_link"
+    number_of_links="10"
+    link_length="0.1"
     link_radius="0.005"
-    link_mass="0.001">
+    link_mass="0.001"
+    load_link_name="${namespace}/load_link">
     <origin xyz="0 0 0" rpy="0 0 0" />
     <inertia ixx="5e-6" ixy="0.0" ixz="0.0" iyy="5e-6" iyz="0.0" izz="5e-6" />
-  </xacro:vertical_cable>
-  <joint name="${namespace}/cable_load_joint" type="fixed">
-    <origin xyz="0 0 -0.5"/>
-    <parent link="${namespace}/cable_link_0b" />
-    <child link="${namespace}/cable_load_link" />
-  </joint>
-    <link name="${namespace}/cable_load_link">
+    <link name="${namespace}/load_link">
       <inertial>
         <mass value="0.2"/>
-        <inertia ixx="0.0002" ixy="0.0002" ixz="0.0002" iyy="0.0002" iyz="0.0" izz="0.0002" />
+        <inertia ixx="0.0002" ixy="0.0" ixz="0.0" iyy="0.0002" iyz="0.0" izz="0.0002" />
       </inertial>
       <visual>
@@ -215,3 +210,4 @@
         </collision> -->
     </link>
+  </xacro:suspended_load>
 </robot>

File: rotors_description/urdf/multirotor_base.xacro (robot description, xacro)
@@ -132,9 +132,29 @@
     </gazebo>
   </xacro:macro>
-  <xacro:macro name="vertical_cable" params="robot_namespace parent number_of_links link_length link_radius link_mass start_link:=0 *origin *link_inertia">
-    <joint name="${robot_namespace}/cable_joint_${start_link}a" type="continuous">
+  <xacro:macro name="ball_joint" params="robot_namespace name parent child damping:=0.0 *origin">
+    <joint name="${robot_namespace}/${name}_aux" type="continuous">
       <xacro:insert_block name="origin" />
       <axis xyz="1 0 0" />
-      <!-- <dynamics damping="0.01"/> -->
+      <dynamics damping="${damping}"/>
+      <parent link="${parent}" />
+      <child link="${robot_namespace}/${name}_link" />
+    </joint>
+    <link name="${robot_namespace}/${name}_link">
+      <inertial>
+        <mass value="${1e-5}"/>
+        <inertia ixx="1e-10" ixy="0" ixz="0" iyy="1e-10" iyz="0" izz="1e-10" />
+      </inertial>
+    </link>
+    <joint name="${robot_namespace}/${name}" type="continuous">
+      <axis xyz="0 1 0" />
+      <dynamics damping="${damping}"/>
+      <parent link="${robot_namespace}/${name}_link" />
+      <child link="${child}" />
+    </joint>
+  </xacro:macro>
+  <xacro:macro name="suspended_load" params="robot_namespace parent number_of_links link_length link_radius link_mass start_link:=0 load_link_name *origin *link_inertia *load_link">
+    <!-- <joint name="${robot_namespace}/cable_joint_${start_link}a" type="continuous">
+      <xacro:insert_block name="origin" />
+      <axis xyz="1 0 0" />
       <parent link="${parent}" />
       <child link="${robot_namespace}/cable_link_${start_link}a" />
@@ -150,7 +170,10 @@
       <parent link="${robot_namespace}/cable_link_${start_link}a" />
       <child link="${robot_namespace}/cable_link_${start_link}b" />
-      <!-- <dynamics damping="0.01"/> -->
-    </joint>
-    <link name="${robot_namespace}/cable_link_${start_link}b">
+    </joint> -->
+    <xacro:ball_joint robot_namespace="${robot_namespace}" name="cable_joint_${start_link}"
+                      parent="${parent}" child="${robot_namespace}/cable_link_${start_link}">
+      <xacro:insert_block name="origin"/>
+    </xacro:ball_joint>
+    <link name="${robot_namespace}/cable_link_${start_link}">
       <origin xyz="0 0 ${-link_length/2}"/>
       <inertial>
@@ -164,24 +187,37 @@
         </geometry>
       </visual>
-        <collision>
+        <!-- <collision>
           <geometry>
             <cylinder length="${link_length}" radius="${link_radius}"/>
           </geometry>
-        </collision>
-    </link>
-    <!-- <xacro:if value="${number_of_links > 1}">
-        <xacro:cable
+        </collision> -->
+    </link>
+    <xacro:if value="${number_of_links > 1}">
+        <xacro:suspended_load
           robot_namespace="${robot_namespace}"
-          suffix="${suffix}"
+          parent="${robot_namespace}/cable_link_${start_link}"
           number_of_links="${number_of_links-1}"
           link_length="${link_length}"
           link_radius="${link_radius}"
           link_mass="${link_mass}"
-          <origin xyz="0 ${arm_length} ${rotor_offset_top}" rpy="0 0 0" />
-          xacro:insert_block name="rotor_inertia" />
-          *origin="${robot_namespace}"
-          *link_inertia="${robot_namespace}"
-          start_link="${start_link+1}" />
-    </xacro:if> -->
+          load_link_name="${load_link_name}"
+          start_link="${start_link+1}" >
+          <origin xyz="0 0 ${-link_length}" />
+          <xacro:insert_block name="link_inertia" />
+          <xacro:insert_block name="load_link" />
+        </xacro:suspended_load>
+    </xacro:if>
+    <xacro:unless value="${number_of_links > 1}">
+      <xacro:ball_joint robot_namespace="${robot_namespace}" name="load_cable_joint"
+                      parent="${robot_namespace}/cable_link_${start_link}" child="${load_link_name}">
+        <origin xyz="0 0 ${-link_length}"/>
+      </xacro:ball_joint>
+      <!-- <joint name="${namespace}/cable_load_joint" type="fixed">
+        <origin xyz="0 0 ${-link_length}"/>
+        <parent link="${robot_namespace}/cable_link_${start_link}b" />
+        <child link="${load_link_name}" />
+      </joint> -->
+      <xacro:insert_block name="load_link" />
+    </xacro:unless>
   </xacro:macro>
 </robot>
